File: squeeki-kleen Video FC.kicad_sch (KiCad schematic)
At the start: 13 parts, among them J1 VCC, J2 VOUT, J3 GND, J4 Conn_Coaxial, Q1 MMBT3906

Commit message: Eevitronics modifications: replace MMCX with solder-wire pads, add fab outputs
See CHANGES.md for the full list of changes (TAPR OHL section 4.2).

Co-Authored-By: Claude Opus 5.5 <noreply@anthropic.com>
Parts:
- removed J4: Conn_Coaxial, Connector_Coaxial:MMCX_Molex_73415-0961_Horizontal_0.8mm-PCB, symbol Connector:Conn_Coaxial
- added J4: Conn_01x02, Connector_Wire:SolderWire-0.25sqmm_1x02_P4.2mm_D0.65mm_OD1.7mm, symbol Connector_Generic:Conn_01x02
- C3, C4: value ~ -> (none)
Connections:
- net CVBS: now also J4.1 (Pin_1)
- net GND: now also J4.2 (Pin_2)
